Commit message: update for Tim

File: realsense2_description/urdf/_d435.front.gazebo.xacro (robot description, xacro)
@@ -6,5 +6,5 @@
 -->
 <robot xmlns:xacro="http://ros.org/wiki/xacro">
-  <xacro:macro name="gazebo_d435_back" params="camera_name reference_link topics_ns depth_optical_frame color_optical_frame infrared1_optical_frame infrared2_optical_frame" >
+  <xacro:macro name="gazebo_d435_front" params="camera_name reference_link topics_ns depth_optical_frame color_optical_frame infrared1_optical_frame infrared2_optical_frame" >
     <!-- Load parameters to model's main link-->
     <xacro:property name="deg_to_rad" value="0.01745329251994329577" />
